File: BCI_chip_PCB/BCI_chip_PCB.kicad_pcb (KiCad board)
At the start: 4 copper layers, 100 x 100 mm, 27 parts, among them J1 225-PRS15001-12, J2 PJ-102AH, J3 A79623-001, U2 SN65LVDS33D, U4 SN65LVDS33D

Commit message: Add updated board
Parts:
- removed C13: 100n, Capacitor_SMD:C_0603_1608Metric
- removed C14: 10u, Capacitor_SMD:C_0603_1608Metric
- removed U4: SN65LVDS33D, avlsi_preferred_parts:D16
- added C10: 100n, Capacitor_SMD:C_0603_1608Metric, F.Cu at (164.0, 95.0)
- added C9: 100n, Capacitor_SMD:C_0603_1608Metric, F.Cu at (157.9, 84.4)
- added U3: SN65LVDS33D, avlsi_preferred_parts:D16, F.Cu at (158.4, 146.2)
- C1: value 10p -> 100n
- C11: value 100n -> 10u
- C2: value 1n -> 10u
- C6: value 1n -> 10p
- C7: value 100n -> 1n
- C8: value 10u -> 1n
- J1: value 225-PRS15001-12 -> A79623-001; footprint avlsi_preferred_parts:225PRS1500112 -> avlsi_preferred_parts:CONN_A79623-001_OMN
- J2: value PJ-102AH -> 225-PRS15001-12; footprint Connector_BarrelJack:BarrelJack_CUI_PJ-102AH_Horizontal -> avlsi_preferred_parts:225PRS1500112
- J3: value A79623-001 -> PJ-102AH; footprint avlsi_preferred_parts:CONN_A79623-001_OMN -> Connector_BarrelJack:BarrelJack_CUI_PJ-102AH_Horizontal
- R2, R3, R4: value 10k -> 100
- R7, R8, R9: value 100 -> 10k
- U1: value ~ -> SN65LVDS33D; footprint avlsi_preferred_parts:avlsi_power_board_opal_kelly -> avlsi_preferred_parts:D16
- U2: value SN65LVDS33D -> ~; footprint avlsi_preferred_parts:D16 -> avlsi_preferred_parts:avlsi_power_board_opal_kelly
- moved U2 106.6 mm to (88.6, 88.4)
- moved J3 75.2 mm to (98.9, 120.3), turned to 0 degrees
- moved J2 58.2 mm to (68.0, 102.0)
- moved J1 54.8 mm to (116.3, 132.3)
- moved C8 51.5 mm to (164.0, 93.3)
- moved C7 50.9 mm to (157.9, 82.8)
- moved C6 50.0 mm to (164.0, 91.6)
- moved C5 48.8 mm to (157.9, 81.2)
- moved C11 42.7 mm to (157.9, 86.0), turned to 0 degrees
- moved U1 40.9 mm to (116.6, 121.5), turned to -90 degrees
- moved C2 32.2 mm to (150.3, 107.9)
- moved C3 32.2 mm to (150.3, 110.4)
- moved C1 32.2 mm to (150.3, 105.4)
- moved C4 32.2 mm to (150.3, 112.9)
- moved C12 28.6 mm to (164.0, 96.6)
Connections:
- C1 pad 1: /VDD08 -> /VCCD33
- C11 pad 1: /VCCD33 -> /VDD08
- C12 pad 1: /VCCD33 -> /VDD08
- C2 pad 1: /VDD08 -> /VCCD33
- C3 pad 1: /VDD08 -> /VCCD33
- C4 pad 1: /VDD08 -> /VCCD33
- J3 pad 1: /NCS_P -> /VDD08
- J3 pad 2: /NCS_N -> /GND
- J3 pad 3: /SCLK_P -> /GND
- R1 pad 2: Net-(U2-G) -> Net-(U1-G)
- R2 pad 1: Net-(U2-*G) -> /NCS_P
- R2 pad 2: /GND -> /NCS_N
- R3 pad 1: /VCCD33 -> /SCLK_P
- R3 pad 2: Net-(U4-G) -> /SCLK_N
- R4 pad 1: Net-(U4-*G) -> /MOSI_P
- R4 pad 2: /GND -> /MOSI_N
- R5 pad 1: /SCLK_P -> /MISO1_P
- R5 pad 2: /SCLK_N -> /MISO1_N
- R6 pad 1: /MOSI_P -> /MISO2_P
- R6 pad 2: /MOSI_N -> /MISO2_N
- R7 pad 1: /NCS_P -> Net-(U1-*G)
- R7 pad 2: /NCS_N -> /GND
- R8 pad 1: /MISO1_P -> /VCCD33
- R8 pad 2: /MISO1_N -> Net-(U3-G)
- R9 pad 1: /MISO2_P -> Net-(U3-*G)
- R9 pad 2: /MISO2_N -> /GND
- U1 pad 10: unconnected-(U1A-FGPA_TDI-Pad10) -> /MISO1_P
- U1 pad 11: /NCS -> /MISO1
- U1 pad 12: unconnected-(U1A-SYS_CLK_MC2-Pad12) -> Net-(U1-*G)
- U1 pad 13: unconnected-(U1A-FPGA_GND-Pad13) -> /MISO2
- U1 pad 14: unconnected-(U1A-FPGA_GND-Pad14) -> /MISO2_P
- U1 pad 15: unconnected-(U1A-MC2_16-Pad15) -> /MISO2_N
- U1 pad 16: unconnected-(U1A-MC2_15_PIN-Pad16) -> /VCCD33
- U2 pad 10: /MISO1_P -> unconnected-(U2A-FGPA_TDI-Pad10)
- U2 pad 11: /MISO1 -> unconnected-(U2A-MC2_12-Pad11)
- U2 pad 12: Net-(U2-*G) -> unconnected-(U2A-SYS_CLK_MC2-Pad12)
- U2 pad 13: /NCS -> unconnected-(U2A-FPGA_GND-Pad13)
- U2 pad 14: /NCS_P -> unconnected-(U2A-FPGA_GND-Pad14)
- U2 pad 15: /NCS_N -> unconnected-(U2A-MC2_16-Pad15)
- U2 pad 16: /VCCD33 -> unconnected-(U2A-MC2_15_PIN-Pad16)
Routing:
- net /ibex_GPIO_OUT_data_o_3_cell: track 0.00 -> 62.7 mm
- net /ibex_GPIO_OUT_data_o_0_cell: track 0.00 -> 60.9 mm
- net /ibex_GPIO_OUT_data_o_4_cell: track 0.00 -> 58.5 mm
- net /ibex_GPIO_OUT_data_o_7_cell: track 0.00 -> 57.3 mm, vias 0 -> 1
- net /ibex_GPIO_OUT_data_o_1_cell: track 0.00 -> 57.2 mm
- net /HALO_clk_rc_i_cell: track 0.00 -> 56.4 mm, vias 0 -> 2
- net /HALO_din_vld_i_cell: track 0.00 -> 55.8 mm, vias 0 -> 2
- net /AMC_sram_mux_i_0_cell: track 0.00 -> 55.1 mm
- net /ibex_GPIO_OUT_data_o_2_cell: track 0.00 -> 51.7 mm
- net /HALO_dout_vld_o_cell: track 0.00 -> 51.3 mm
- net /HALO_clk_lic_i_cell: track 0.00 -> 51.0 mm, vias 0 -> 2
- net /AMC_sram_error_o_cell: track 0.00 -> 50.8 mm
- net /AMC_sram_finish_o_cell: track 0.00 -> 49.8 mm
- net /HALO_cfg_sel_i_cell: track 0.00 -> 48.4 mm
- net /HALO_clk_aes_i_cell: track 0.00 -> 48.4 mm, vias 0 -> 2
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Other:
- board text added: "BCI Test Board Rev. 1 Thomas Jagielski AVLSI LAB"
- board text added: "VCCD09"
- board text added: "VCCD12"
- board text added: "VCCD18"
- board text added: "VCCD25"
- board text added: "VCCD33"
- board text added: "VDCustom"
- board text added: "VDIN5"
- board text removed: "Brain Computer Interface (BCI) Test Board Rev. 1"
