File: BCI_chip_PCB/BCI_chip_PCB.kicad_sch (KiCad schematic)
At the start: 27 parts, among them J1 225-PRS15001-12, J2 PJ-102AH, J3 A79623-001, U2 SN65LVDS33D, U4 SN65LVDS33D

Commit message: Add updated board
Parts:
- renumbered C13 to C1, C3 to C10, C8 to C11, C4 to C12, C14 to C2, C11 to C3, C12 to C4, C1 to C6, C6 to C7, C2 to C8, C7 to C9, J3 to J1, J1 to J2, J2 to J3, R7 to R2, R5 to R3, R6 to R4, R8 to R5, R9 to R6, R2 to R7, R3 to R8, R4 to R9, U2 to U1, U1 to U2, U4 to U3
Connections:
- net AMC_sram_error_o_cell: now also U2.78 (MC2_77_PIN)
- net AMC_sram_finish_o_cell: now also U2.80 (MC2_79_PIN)
- net AMC_sram_mux_i_0_cell: now also U2.73 (MC2_74_PIN)
- net AMC_sram_mux_i_1_cell: now also U2.139 (MC1_60_PIN)
- net AMC_sram_mux_i_2_cell: now also U2.137 (MC1_58_PIN)
- net AMC_sram_reset_i_cell: now also U2.75 (MC2_76_PIN)
- net AMC_sram_sleep_i_cell: now also U2.133 (MC1_54_PIN)
- net AMC_sram_test_i_cell: now also U2.71 (MC2_72_PIN)
- net GND: now also J2.D15, U2.176 (DGND), U2.178 (DGND), U2.180 (DGND), U2.182 (DGND), U2.184 (DGND), U2.186 (DGND), U2.188 (DGND); no longer U2.190 (DGND), U2.192 (DGND), U2.194 (DGND), U2.196 (DGND), U2.198 (DGND), U2.200 (DGND), U2.202 (DGND), U2.204 (DGND), U2.206 (DGND), U2.208 (DGND), U2.210 (DGND), U2.212 (DGND), U2.214 (DGND), U2.216 (DGND)
- net HALO_aes_en_i_cell: now also U2.130 (MC1_49_PIN)
- net HALO_cfg_ack_o_cell: now also U2.64 (MC2_63_PIN)
- net HALO_cfg_data_in_i_cell: now also U2.51 (MC2_52_PIN)
- net HALO_cfg_data_in_valid_i_cell: now also U2.49 (MC2_50_PIN)
- net HALO_cfg_data_out_o_cell: now also U2.68 (MC2_67_PIN)
- net HALO_cfg_en_i_cell: now also U2.57 (MC2_58_PIN)
- net HALO_cfg_mux_i_0_cell: now also U2.34 (MC2_33_PIN)
- net HALO_cfg_mux_i_1_cell: now also U2.99 (MC1_20_PIN)
- net HALO_cfg_mux_i_2_cell: now also U2.119 (MC1_40_PIN)
- net HALO_cfg_mux_i_3_cell: now also U2.42 (MC2_41_PIN)
- net HALO_cfg_rw_i_cell: now also U2.61 (MC2_62_PIN)
- net HALO_cfg_sel_i_cell: now also U2.67 (MC2_68_PIN)
- net HALO_clk_aes_i_cell: now also U2.59 (MC2_60_PIN)
- net HALO_clk_dwt_i_cell: now also U2.53 (MC2_54_PIN)
- net HALO_clk_gate_i_cell: now also U2.43 (MC2_44_PIN)
- net HALO_clk_in_i_cell: now also U2.63 (MC2_64_PIN)
- net HALO_clk_in_internal_o_cell: now also U2.62 (MC2_61_PIN)
- net HALO_clk_intcnt_i_cell: now also U2.45 (MC2_46_PIN)
- net HALO_clk_lic_i_cell: now also U2.97 (MC1_18_PIN)
- net HALO_clk_lz_i_cell: now also U2.44 (MC2_43_PIN)
- net HALO_clk_ma_i_cell: now also U2.47 (MC2_48_PIN)
- net HALO_clk_neo_i_cell: now also U2.65 (MC2_66_PIN)
- net HALO_clk_out_i_cell: now also U2.46 (MC2_45_PIN)
- net HALO_clk_out_internal_o_cell: now also U2.66 (MC2_65_PIN)
- net HALO_clk_rc_i_cell: now also U2.101 (MC1_22_PIN)
- net HALO_clk_thr_i_cell: now also U2.38 (MC2_37_PIN)
- net HALO_clk_tok_i_cell: now also U2.103 (MC1_24_PIN)
- net HALO_din_data_i_0_cell: now also U2.113 (MC1_34_PIN)
- net HALO_din_data_i_1_cell: now also U2.107 (MC1_28_PIN)
- net HALO_din_data_i_2_cell: now also U2.109 (MC1_30_PIN)
- net HALO_din_data_i_3_cell: now also U2.111 (MC1_32_PIN)
- net HALO_din_data_i_4_cell: now also U2.117 (MC1_38_PIN)
- net HALO_din_data_i_5_cell: now also U2.121 (MC1_42_PIN)
- net HALO_din_data_i_6_cell: now also U2.124 (MC1_43_PIN)
- net HALO_din_data_i_7_cell: now also U2.120 (MC1_39_PIN)
- net HALO_din_vld_i_cell: now also U2.95 (MC1_16_PIN)
- net HALO_dout_data_o_0_cell: now also U2.100 (MC1_19_PIN)
- net HALO_dout_data_o_1_cell: now also U2.102 (MC1_21_PIN)
- net HALO_dout_data_o_2_cell: now also U2.104 (MC1_23_PIN)
- net HALO_dout_data_o_3_cell: now also U2.106 (MC1_25_PIN)
- net HALO_dout_data_o_4_cell: now also U2.72 (MC2_71_PIN)
- net HALO_dout_data_o_5_cell: now also U2.70 (MC2_69_PIN)
- net HALO_dout_data_o_6_cell: now also U2.74 (MC2_73_PIN)
- net HALO_dout_data_o_7_cell: now also U2.76 (MC2_75_PIN)
- net HALO_dout_vld_o_cell: now also U2.96 (MC1_15_PIN)
- net HALO_gate_en_i_cell: now also U2.129 (MC1_50_PIN)
- net HALO_pipeline_i_0_cell: now also U2.126 (MC1_45_PIN)
- net HALO_pipeline_i_1_cell: now also U2.134 (MC1_53_PIN)
- net HALO_pipeline_i_2_cell: now also U2.132 (MC1_51_PIN)
- net HALO_pipeline_i_3_cell: now also U2.131 (MC1_52_PIN)
- net HALO_rst_ni_cell: now also U2.69 (MC2_70_PIN)
- net HALO_top_mux_i_cell: now also U2.105 (MC1_26_PIN)
- net NCS: now also U2.152 (MC1_71); no longer U2.11 (MC2_12)
- net VCCD33: now also U2.185 (VCCD33); no longer U2.199 (VCCD33), U2.213 (VCCD33)
- net VDD08: now also U2.175 (VDCustom); no longer U2.189 (VDCustom), U2.203 (VDCustom)
- net ibex_GPIO_OUT_data_o_0_cell: now also U2.58 (MC2_57_PIN)
- net ibex_GPIO_OUT_data_o_1_cell: now also U2.52 (MC2_51_PIN)
- net ibex_GPIO_OUT_data_o_2_cell: now also U2.48 (MC2_47_PIN)
- net ibex_GPIO_OUT_data_o_3_cell: now also U2.60 (MC2_59_PIN)
- net ibex_GPIO_OUT_data_o_4_cell: now also U2.54 (MC2_53_PIN)
- net ibex_GPIO_OUT_data_o_5_cell: now also U2.28 (MC2_27_PIN)
- net ibex_GPIO_OUT_data_o_6_cell: now also U2.30 (MC2_29_PIN)
- net ibex_GPIO_OUT_data_o_7_cell: now also U2.50 (MC2_49_PIN)
- net ibex_GPIO_OUT_valid_o_cell: now also U2.98 (MC1_17_PIN)
- net ibex_SPI_slave_MOSI_i_cell: now also U2.128 (MC1_47_PIN)
- net ibex_SPI_slave_SCLK_i_cell: now also U2.127 (MC1_48_PIN)
- net ibex_clk_i_cell: now also U2.40 (MC2_39_PIN)
- net ibex_irq_i_cell: now also U2.123 (MC1_44_PIN)
- net ibex_prog_i_cell: now also U2.125 (MC1_46_PIN)
- net ibex_rst_ni_cell: now also U2.122 (MC1_41_PIN)
- no-connect marks 75 -> 79
Other:
- note added: "Level Shifter 1 Port A Input to Chip"
- note added: "Level Shifter 1 Port B Input to Chip"
- note added: "Level Shifter 2 Port A Output from Chip"
- note added: "Level Shifter 2 Port B Input to Chip"
- note added: "Level Shifter 3 Port A Input to Chip"
- note added: "Level Shifter 4 Port A Input from Chip"
- note added: "Level Shifter 4 Port B Input from Chip"
- note added: "Level Shifter 4 Port B Output from Chip"
- note added: "Level Shifter 5 Port A Input from Chip"
- note added: "Level Shifter 5 Port A Output from Chip"
- note added: "Level Shifter 6 Port A Ouput from Chip"
- note added: "Level Shifter 6 Port B Output from Chip"
- moved on the sheet: U2B
